File: cc2650_simplified.brd (EAGLE design)
At the start: 50.5 x 22.9 mm, 13 parts, among them IC4 CC2650MODAMOHR, U402 TPS62233DRY

Commit message: board size, gerber files
Other:
- board size 50.5 x 22.9 mm -> 50.7 x 23.1 mm
- board text added: "Rev A"
- board text added: "Team Rocket"
Changed lines of the file:
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@@
 <board>
 <plain>
-<wire x1="0" y1="0" x2="50.47" y2="0" width="0" layer="20"/>
-<wire x1="50.47" y1="0" x2="50.47" y2="22.85" width="0" layer="20"/>
-<wire x1="50.47" y1="22.85" x2="0" y2="22.85" width="0" layer="20"/>
+<wire x1="0" y1="0" x2="50.72" y2="-0.25" width="0" layer="20"/>
+<wire x1="50.72" y1="-0.25" x2="50.72" y2="22.6" width="0" layer="20"/>
+<wire x1="50.72" y1="22.6" x2="0" y2="22.85" width="0" layer="20"/>
 <wire x1="0" y1="22.85" x2="0" y2="0" width="0" layer="20"/>
 <dimension x1="0" y1="0" x2="50.8" y2="0" x3="25.4" y3="-3.81" textsize="1.778" layer="1"/>
@@
 <hole x="48.5" y="21" drill="1"/>
 <hole x="2" y="21" drill="1"/>
+<text x="3" y="8" size="1.778" layer="1">Team Rocket</text>
+<text x="3" y="8" size="1.778" layer="1">Team Rocket</text>
+<text x="4" y="8" size="1.778" layer="1">Team Rocket</text>
+<text x="4" y="8" size="1.778" layer="1">Team Rocket</text>
+<text x="3" y="9" size="1.016" layer="21">Team Rocket</text>
+<text x="3" y="7" size="1.016" layer="21">Rev A</text>
 </plain>
 <attributes>
