File: cc2650_48.sch (EAGLE design)
At the start: 21 parts, among them IC1 CC2650F128RGZT, SW1 SPST_TACT-KMR2, SW2 SPST_TACT-KMR2, U402 TPS62233DRY, X3 microUSB

Commit message: added 48 pin cc2650. change res, cap, led to bigger packages. moved battery to bottom of board. changed micro usb.
Parts:
- removed LED3: (no value), led:LEDCHIP-LED0603
- added LED1: (no value), led:LEDCHIPLED_0805
Connections:
- net GND: now also LED1.C; no longer LED3.C
- net N$32: now also LED1.A; no longer LED3.A
Changed lines of the file:
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@@
 <part name="GND7" library="supply1" deviceset="GND" device=""/>
 <part name="GND21" library="supply1" deviceset="GND" device=""/>
-<part name="LED3" library="led" library_urn="urn:adsk.eagle:library:259" deviceset="LED" device="CHIP-LED0603" package3d_urn="urn:adsk.eagle:package:15819/1">
-<attribute name="MF" value=""/>
-<attribute name="MPN" value="HSME-C191"/>
-<attribute name="OC_NEWARK" value="05M0345"/>
-</part>
 <part name="GND64" library="supply1" deviceset="GND" device=""/>
 <part name="U402" library="tps62231dry" deviceset="TPS6223X_DRY_6" device="" value="TPS62233DRY">
@@
 <part name="C10" library="adafruit" deviceset="C-US" device="C0805" value="1n"/>
 <part name="IC1" library="CC2650F128RGZT" deviceset="CC2650F128RGZT" device=""/>
+<part name="LED1" library="led" library_urn="urn:adsk.eagle:library:259" deviceset="LED" device="CHIPLED_0805" package3d_urn="urn:adsk.eagle:package:15821/1"/>
 </parts>
 <sheets>
@@
 <instance part="GND7" gate="1" x="45.72" y="50.8"/>
 <instance part="GND21" gate="1" x="154.94" y="60.96"/>
-<instance part="LED3" gate="G$1" x="139.7" y="68.58" rot="R90">
-<attribute name="OC_NEWARK" x="139.7" y="68.58" size="1.778" layer="96" display="off"/>
-<attribute name="MF" x="139.7" y="68.58" size="1.778" layer="96" display="off"/>
-<attribute name="MPN" x="139.7" y="68.58" size="1.778" layer="96" display="off"/>
-</instance>
 <instance part="GND64" gate="1" x="76.2" y="-15.24"/>
 <instance part="U402" gate="&gt;NAME" x="139.7" y="7.62">
@@
 <instance part="C10" gate="G$1" x="45.72" y="63.5"/>
 <instance part="IC1" gate="G$1" x="-193.04" y="15.24"/>
+<instance part="LED1" gate="G$1" x="139.7" y="68.58" rot="R90"/>
 </instances>
 <busses>
@@
 </segment>
 <segment>
-<pinref part="LED3" gate="G$1" pin="C"/>
 <pinref part="GND21" gate="1" pin="GND"/>
 <wire x1="144.78" y1="68.58" x2="154.94" y2="68.58" width="0.1524" layer="91"/>
 <wire x1="154.94" y1="68.58" x2="154.94" y2="63.5" width="0.1524" layer="91"/>
-<junction x="144.78" y="68.58"/>
 <junction x="154.94" y="63.5"/>
+<pinref part="LED1" gate="G$1" pin="C"/>
 </segment>
 <segment>
@@
 <segment>
 <wire x1="137.16" y1="68.58" x2="134.62" y2="68.58" width="0.1524" layer="91"/>
-<pinref part="LED3" gate="G$1" pin="A"/>
-<junction x="137.16" y="68.58"/>
 <pinref part="R6" gate="G$1" pin="2"/>
-</segment>
-</net>
+<pinref part="LED1" gate="G$1" pin="A"/>
+</segment>
+</net>
